File: hardware/ws2812-clock.kicad_sch (KiCad schematic)
At the start: 31 parts, among them J1 Conn_01x01_Pin, Q3 2N7002, SW2 Reset ESP, SW5 Toggle AP, SW6 Toggle Alarm, SW7 Snooze Alarm, U1 ESP32-WROOM-32D, U3 SHT30-DIS, U4 AMS1117-3.3, U5 DMP3026SFDE-7

Commit message: Updated PCB
Parts:
- removed U5: DMP3026SFDE-7, reverse_polarity_diode:U-DFN2020-6E_L2.0-W2.0-P0.65-BL, symbol reverse_polarity_diode:DMP3026SFDE-7
- added C245: 100n, Capacitor_SMD:C_0402_1005Metric, symbol Device:C_Small
- added Q5: AO4485, reverse_polarity_diode:SOIC-8_L5.0-W4.0-P1.27-LS6.0-BL, symbol reverse_polarity_diode:AO4485
- added U5: BME280, bme280:LGA-8_BME280_BL, symbol bme280:BME280
- J1: LCSC (none) -> DNP
Connections:
- net +3.3V: now also C245.1, U5.2 (CSB), U5.6 (VDDIO), U5.8 (VDD)
- net +5V: now also Q5.2 (S)
- net GND: now also C245.2, Q5.4 (G), U5.1 (GND), U5.5 (SDO), U5.7 (GND)
- net SCL: now also U5.4 (SCK)
- net SDA: now also U5.3 (SDI)
- net at DC1.1, JP2.2 (B): now also Q5.6 (D)
Other:
- moved on the sheet: C240, DC1, JP1, JP2, U3

Commit message: Update mosfet circuit
Connections:
- net +5V: now also Q5.1 (S), Q5.3 (S)
- net at DC1.1, JP2.2 (B), Q5.6 (D): now also Q5.5 (D), Q5.7 (D)
Changed lines of the file:
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@@
   (junction (at 191.135 64.77) (diameter 0) (color 0 0 0 0)
   )
+  (junction (at 131.445 35.56) (diameter 0) (color 0 0 0 0)
+  )
   (junction (at 160.655 64.77) (diameter 0) (color 0 0 0 0)
   )
@@
   (junction (at 133.985 155.575) (diameter 0) (color 0 0 0 0)
   )
+  (junction (at 146.685 33.02) (diameter 0) (color 0 0 0 0)
+  )
+  (junction (at 146.685 35.56) (diameter 0) (color 0 0 0 0)
+  )
   (junction (at 123.19 94.615) (diameter 0) (color 0 0 0 0)
   )
@@
   )
   (junction (at 128.27 75.565) (diameter 0) (color 0 0 0 0)
+  )
+  (junction (at 131.445 33.02) (diameter 0) (color 0 0 0 0)
   )
   (junction (at 128.905 33.02) (diameter 0) (color 0 0 0 0)
@@
     (stroke (width 0) (type default))
   )
+  (wire (pts (xy 131.445 33.02) (xy 131.445 35.56))
+    (stroke (width 0) (type default))
+  )
   (wire (pts (xy 123.19 99.695) (xy 135.89 99.695))
     (stroke (width 0) (type default))
@@
     (stroke (width 0) (type default))
   )
+  (wire (pts (xy 146.685 33.02) (xy 146.685 35.56))
+    (stroke (width 0) (type default))
+  )
   (wire (pts (xy 111.76 115.57) (xy 125.73 115.57))
     (stroke (width 0) (type default))
@@
     (stroke (width 0) (type default))
   )
+  (wire (pts (xy 131.445 35.56) (xy 131.445 38.1))
+    (stroke (width 0) (type default))
+  )
   (wire (pts (xy 155.575 71.12) (xy 155.575 72.39))
     (stroke (width 0) (type default))
@@
     (stroke (width 0) (type default))
   )
+  (wire (pts (xy 146.685 35.56) (xy 146.685 38.1))
+    (stroke (width 0) (type default))
+  )

Commit message: Fixed PCB trace
Connections:
- net leds/LED_DATA_IN: now also U1.8 (IO32); no longer U1.6 (IO34)
Changed lines of the file:
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@@
   (no_connect (at 54.61 75.565))
   (no_connect (at 85.09 93.345))
-  (no_connect (at 85.09 90.805))
+  (no_connect (at 85.09 95.885))
   (no_connect (at 85.09 45.085))
   (no_connect (at 85.09 85.725))
@@
     (stroke (width 0) (type default))
   )
-  (wire (pts (xy 85.09 95.885) (xy 89.535 95.885))
-    (stroke (width 0) (type default))
-  )
   (wire (pts (xy 179.07 98.425) (xy 179.07 109.22))
     (stroke (width 0) (type default))
@@
   )
   (wire (pts (xy 155.575 64.77) (xy 155.575 66.04))
+    (stroke (width 0) (type default))
+  )
+  (wire (pts (xy 85.09 90.805) (xy 88.9 90.805))
     (stroke (width 0) (type default))
   )
@@
     )
   )
-  (sheet (at 89.535 93.98) (size 26.035 3.81) (fields_autoplaced)
+  (sheet (at 88.9 88.9) (size 26.035 3.81) (fields_autoplaced)
     (stroke (width 0.1524) (type solid))
     (fill (color 0 0 0 0.0000))
-    (property "Sheetname" "leds" (at 89.535 93.2684 0)
+    (property "Sheetname" "leds" (at 88.9 88.1884 0)
       (effects (font (size 1.27 1.27)) (justify left bottom))
     )
-    (property "Sheetfile" "leds.kicad_sch" (at 89.535 98.3746 0)
+    (property "Sheetfile" "leds.kicad_sch" (at 88.9 93.2946 0)
       (effects (font (size 1.27 1.27)) (justify left top))
     )
-    (pin "LED_DATA_IN" input (at 89.535 95.885 180)
-      (effects (font (size 1.27 1.27)) (justify left))
-    )
+    (pin "LED_DATA_IN" input (at 88.9 90.805 180)
+      (effects (font (size 1.27 1.27)) (justify left))
+    )

Commit message: More fixes
Parts:
- added TP1, TP2, TP3: TestPoint_Probe, TestPoint:TestPoint_Pad_D2.0mm, symbol Connector:TestPoint_Probe
Connections:
- net SCL: now also U1.11 (IO26), TP2.1; no longer U1.22 (SDI/SD1)
- net SDA: now also U1.10 (IO25), TP1.1; no longer U1.21 (SDO/SD0)
- net leds/LED_DATA_IN renamed LEDS
- net LEDS: now also TP3.1
Changed lines of the file:
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@@
   (junction (at 191.135 72.39) (diameter 0) (color 0 0 0 0)
   )
+  (junction (at 92.075 90.805) (diameter 0) (color 0 0 0 0)
+  )
   (junction (at 69.85 26.67) (diameter 0) (color 0 0 0 0)
   )
@@
   )
   (no_connect (at 85.09 88.265))
+  (no_connect (at 54.61 70.485))
   (no_connect (at 54.61 78.105))
   (no_connect (at 85.09 70.485))
-  (no_connect (at 85.09 83.185))
   (no_connect (at 85.09 73.025))
   (no_connect (at 54.61 47.625))
+  (no_connect (at 54.61 73.025))
   (no_connect (at 85.09 52.705))
   (no_connect (at 54.61 83.185))
@@
   (no_connect (at 85.09 95.885))
   (no_connect (at 85.09 45.085))
-  (no_connect (at 85.09 85.725))
   (wire (pts (xy 123.19 89.535) (xy 123.19 94.615))
     (stroke (width 0) (type default))
   )
+  (wire (pts (xy 85.09 83.185) (xy 86.995 83.185))
+    (stroke (width 0) (type default))
+  )
   (wire (pts (xy 85.09 57.785) (xy 88.265 57.785))
     (stroke (width 0) (type default))
@@
     (stroke (width 0) (type default))
   )
+  (wire (pts (xy 183.515 29.845) (xy 186.69 29.845))
+    (stroke (width 0) (type default))
+  )
   (wire (pts (xy 121.285 120.65) (xy 121.285 125.73))
     (stroke (width 0) (type default))
@@
     (stroke (width 0) (type default))
   )
+  (wire (pts (xy 85.09 85.725) (xy 86.995 85.725))
+    (stroke (width 0) (type default))
+  )
   (wire (pts (xy 179.07 109.22) (xy 179.07 119.38))
     (stroke (width 0) (type default))
@@
     (stroke (width 0) (type default))
   )
+  (wire (pts (xy 183.515 34.925) (xy 186.69 34.925))
+    (stroke (width 0) (type default))
+  )
   (wire (pts (xy 86.995 75.565) (xy 85.09 75.565))
     (stroke (width 0) (type default))
@@
     (stroke (width 0) (type default))
   )
+  (wire (pts (xy 92.075 90.805) (xy 95.25 90.805))
+    (stroke (width 0) (type default))
+  )
   (wire (pts (xy 59.69 27.305) (xy 59.69 26.67))
     (stroke (width 0) (type default))
@@
     (stroke (width 0) (type default))
   )
-  (wire (pts (xy 52.705 73.025) (xy 54.61 73.025))
-    (stroke (width 0) (type default))
-  )
   (wire (pts (xy 157.48 121.285) (xy 157.48 123.19))
     (stroke (width 0) (type default))
@@
     (stroke (width 0) (type default))
   )
-  (wire (pts (xy 85.09 90.805) (xy 88.9 90.805))
+  (wire (pts (xy 85.09 90.805) (xy 92.075 90.805))
+    (stroke (width 0) (type default))
+  )
+  (wire (pts (xy 93.98 85.09) (xy 92.075 85.09))
     (stroke (width 0) (type default))
   )
@@
     (stroke (width 0) (type default))
   )
+  (wire (pts (xy 92.075 85.09) (xy 92.075 90.805))
+    (stroke (width 0) (type default))
+  )
   (wire (pts (xy 59.69 26.67) (xy 62.23 26.67))
     (stroke (width 0) (type default))
@@
     (stroke (width 0) (type default))
   )
-  (wire (pts (xy 52.705 70.485) (xy 54.61 70.485))
-    (stroke (width 0) (type default))
-  )
   (wire (pts (xy 179.07 138.43) (xy 179.07 147.955))
     (stroke (width 0) (type default))
@@
   )
   (wire (pts (xy 124.46 46.355) (xy 128.905 46.355))
+    (stroke (width 0) (type default))
+  )
+  (wire (pts (xy 182.88 40.005) (xy 186.69 40.005))
     (stroke (width 0) (type default))
   )
@@
     (effects (font (size 1.27 1.27)) (justify left bottom))
   )
+  (label "SCL" (at 183.515 34.925 180) (fields_autoplaced)
+    (effects (font (size 1.27 1.27)) (justify right bottom))
+  )
   (label "ESP_RX" (at 60.325 156.21 180) (fields_autoplaced)
     (effects (font (size 1.27 1.27)) (justify right bottom))
@@
     (effects (font (size 1.27 1.27)) (justify left bottom))
   )
+  (label "LEDS" (at 93.98 85.09 0) (fields_autoplaced)
+    (effects (font (size 1.27 1.27)) (justify left bottom))
+  )
   (label "IO0" (at 92.71 40.005 0) (fields_autoplaced)
     (effects (font (size 1.27 1.27)) (justify left bottom))
@@
     (effects (font (size 1.27 1.27)) (justify left bottom))
   )
-  (label "SDA" (at 52.705 70.485 180) (fields_autoplaced)
-    (effects (font (size 1.27 1.27)) (justify right bottom))
-  )
   (label "SNOOZE_ALARM" (at 86.995 80.645 0) (fields_autoplaced)
     (effects (font (size 1.27 1.27)) (justify left bottom))
   )
+  (label "SDA" (at 183.515 29.845 180) (fields_autoplaced)
+    (effects (font (size 1.27 1.27)) (justify right bottom))
+  )
   (label "BEEPER" (at 130.175 155.575 180) (fields_autoplaced)
     (effects (font (size 1.27 1.27)) (justify right bottom))
@@
     (effects (font (size 1.27 1.27)) (justify right bottom))
   )
+  (label "LEDS" (at 182.88 40.005 180) (fields_autoplaced)
+    (effects (font (size 1.27 1.27)) (justify right bottom))
+  )
   (label "STA_STATUS_LED" (at 86.995 65.405 0) (fields_autoplaced)
     (effects (font (size 1.27 1.27)) (justify left bottom))
@@
     (effects (font (size 1.27 1.27)) (justify right bottom))
   )
-  (label "SCL" (at 52.705 73.025 180) (fields_autoplaced)
-    (effects (font (size 1.27 1.27)) (justify right bottom))
+  (label "SCL" (at 86.995 85.725 0) (fields_autoplaced)
+    (effects (font (size 1.27 1.27)) (justify left bottom))
+  )
+  (label "SDA" (at 86.995 83.185 0) (fields_autoplaced)
+    (effects (font (size 1.27 1.27)) (justify left bottom))
   )
   (symbol (lib_id "tactile_button:TS-1088R-02026") (at 191.77 138.43 0) (unit 1)
@@
     )
   )
+  (symbol (lib_id "Connector:TestPoint_Probe") (at 186.69 34.925 0) (unit 1)
+    (in_bom yes) (on_board yes) (dnp no) (fields_autoplaced)
+    (property "Reference" "TP2" (at 191.135 32.0675 0)
+      (effects (font (size 1.27 1.27)) (justify left))
+    )
+    (property "Value" "TestPoint_Probe" (at 191.135 34.6075 0)
+      (effects (font (size 1.27 1.27)) (justify left))
+    )
+    (property "Footprint" "TestPoint:TestPoint_Pad_D2.0mm" (at 191.77 34.925 0)
+      (effects (font (size 1.27 1.27)) hide)
+    )
+    (property "Datasheet" "~" (at 191.77 34.925 0)
+      (effects (font (size 1.27 1.27)) hide)
+    )
+    (pin "1")
+    (instances
+      (project "ws2812-clock"
+        (path "/4ccf6c15-bcf8-4d9c-b268-c98587b05c40"
+          (reference "TP2") (unit 1)
+        )
+      )
+    )
+  )
   (symbol (lib_id "Device:C_Small") (at 155.575 68.58 180) (unit 1)
     (in_bom yes) (on_board yes) (dnp no)
@@
         (path "/87b1e95a-e278-444a-acb4-c3f9785f69cd"
           (reference "#PWR0111") (unit 1)
+        )
+      )
+    )
+  )
+  (symbol (lib_id "Connector:TestPoint_Probe") (at 186.69 29.845 0) (unit 1)
+    (in_bom yes) (on_board yes) (dnp no) (fields_autoplaced)
+    (property "Reference" "TP1" (at 191.135 26.9875 0)
+      (effects (font (size 1.27 1.27)) (justify left))
+    )
+    (property "Value" "TestPoint_Probe" (at 191.135 29.5275 0)
+      (effects (font (size 1.27 1.27)) (justify left))
+    )
+    (property "Footprint" "TestPoint:TestPoint_Pad_D2.0mm" (at 191.77 29.845 0)
+      (effects (font (size 1.27 1.27)) hide)
+    )
+    (property "Datasheet" "~" (at 191.77 29.845 0)
+      (effects (font (size 1.27 1.27)) hide)
+    )
+    (pin "1")
+    (instances
+      (project "ws2812-clock"
+        (path "/4ccf6c15-bcf8-4d9c-b268-c98587b05c40"
+          (reference "TP1") (unit 1)
         )
       )
@@
     )
   )
+  (symbol (lib_id "Connector:TestPoint_Probe") (at 186.69 40.005 0) (unit 1)
+    (in_bom yes) (on_board yes) (dnp no) (fields_autoplaced)
+    (property "Reference" "TP3" (at 191.135 37.1475 0)
+      (effects (font (size 1.27 1.27)) (justify left))
+    )
+    (property "Value" "TestPoint_Probe" (at 191.135 39.6875 0)
+      (effects (font (size 1.27 1.27)) (justify left))
+    )
+    (property "Footprint" "TestPoint:TestPoint_Pad_D2.0mm" (at 191.77 40.005 0)
+      (effects (font (size 1.27 1.27)) hide)
+    )
+    (property "Datasheet" "~" (at 191.77 40.005 0)
+      (effects (font (size 1.27 1.27)) hide)
+    )
+    (pin "1")
+    (instances
+      (project "ws2812-clock"
+        (path "/4ccf6c15-bcf8-4d9c-b268-c98587b05c40"
+          (reference "TP3") (unit 1)
+        )
+      )
+    )
+  )
   (symbol (lib_id "Jumper:SolderJumper_2_Open") (at 144.78 49.53 0) (unit 1)
     (in_bom yes) (on_board yes) (dnp no)
@@
     )
   )
-  (sheet (at 88.9 88.9) (size 26.035 3.81) (fields_autoplaced)
+  (sheet (at 95.25 88.9) (size 26.035 3.81) (fields_autoplaced)
     (stroke (width 0.1524) (type solid))
     (fill (color 0 0 0 0.0000))
-    (property "Sheetname" "leds" (at 88.9 88.1884 0)
+    (property "Sheetname" "leds" (at 95.25 88.1884 0)
       (effects (font (size 1.27 1.27)) (justify left bottom))
     )
-    (property "Sheetfile" "leds.kicad_sch" (at 88.9 93.2946 0)
+    (property "Sheetfile" "leds.kicad_sch" (at 95.25 93.2946 0)
       (effects (font (size 1.27 1.27)) (justify left top))
     )
-    (pin "LED_DATA_IN" input (at 88.9 90.805 180)
-      (effects (font (size 1.27 1.27)) (justify left))
-    )
+    (pin "LED_DATA_IN" input (at 95.25 90.805 180)
+      (effects (font (size 1.27 1.27)) (justify left))
+    )

Commit message: PCB rework (ordered)
Parts:
- added J2: Conn_01x04, Connector_PinHeader_2.54mm:PinHeader_1x04_P2.54mm_Vertical, symbol Connector_Generic:Conn_01x04
- added JP3, JP4, JP5: SolderJumper_2_Open, Jumper:SolderJumper-2_P1.3mm_Open_TrianglePad1.0x1.5mm, symbol Jumper:SolderJumper_2_Open
Connections:
- net +3.3V: now also J2.1 (Pin_1)
- net ALARM_STATUS_LED: now also JP5.1 (A); no longer R16.2
- net AP_STATUS_LED: now also JP3.1 (A); no longer R14.2
- net GND: now also J2.4 (Pin_4)
- net SCL: now also J2.3 (Pin_3)
- net SDA: now also J2.2 (Pin_2)
- net STA_STATUS_LED: now also JP4.1 (A); no longer R15.2
- new net: JP3.2 (B), R14.2
- new net: JP5.2 (B), R16.2
- new net: JP4.2 (B), R15.2
Other:
- moved on the sheet: C240, C241, C242, C243, C244, D234, D235, J1, R14, R15, R16, U3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

Commit message: Backup from Macbook
Parts:
- renumbered D234 to D237, D234 to D238, D235 to D239, R5 to R13
